Commit message: [x3_description] several major changes to agent namespacing and Gazebo simulation
Under `urdf`:
- modified existing xacro files for agent namespacing (`x3_body.xacro`, `x3_sensors.xacro`, and `x3.urdf.xacro`)
- added gazebo properties for Gazebo simulation physical parameters (wheel joint friction constant and depth) and sensors (LiDAR and IMU)
- added gazebo control and ros2 control xacro file to permit robot control using either method

Under `worlds`:
- added `empty_world` and `world_1` SDF files from ROS2_DRL_Navigation repo

Under `launch`:
- `display.launch.py`: 1. made agent namespacing effective, 2. added an argument to control whether to use rviz visualization only (to use with Gazebo or real world deployment, where robot state and joint state publishers are already taken care of)
- added `gazebo.launch.py`, `launch_odom.py`, and `launch_world.py` to launch the Gazebo simulation. Handled several problems related to agent spawning, OdometryPublisher odom offset, multiple sources of tf fighting one another

Under `config` - added configuration for Gazebo sim, ros2_control, and ekf filter
- added `controllers.yaml` as a placeholder default for ros2_contro. Added `controllers.yaml.template` with `__AGENT_NAME__` placeholder, which is rendered when launching gazebo to have it replaced with the agent_name runtime argument
- added `ekf_params` YAML file with $(var agent_name) to handle agent name spacing of different frames, different sources of odometry input data which are all namespaced under the agent_name on rqt_graph
- added `gz_bridge_gazebo_control` to bridge between gazebo ign topics and ROS2 topics when using gazebo control
- added `gz_bridge_ros2_control` YAML to bridge between gazebo ign topics and ROS2 topic when using ros2_control (tf is currently commented due to a problem where OdometryPublisher plugin is unaware of different robot agent spawn locations in Gazebo and keeps the odom frame stuck at world origin)

under `x3_description`:
- added `odom_offset_node` to handle the offset when using the odometry odom_OP published by the OdometryPublisher plugin (unaware of initial agent spawn location offset) => this node handles the static shift in the odometry offset to turn from /<agent_name>/odom_OP to the desired /<agent_name>/odom topic
- added `odom_to_vel_raw` node, which subscribes to the wheel odometry published by the ros2 control plugin (diff drive controller odometry) and publishes the TwistStamped portion of this message for EKF odometry fusion (twist0)

File: src/x3_description/urdf/x3.urdf.xacro (robot description, xacro)
@@ -1,7 +1,14 @@
 <?xml version = "1.0"?>
 <robot name = "agent" xmlns:xacro = "http://www.ros.org/wiki/xacro">
-    <!-- ========== Common Macros ========== -->
-    <xacro:macro name="common_link" params="name material *origin collision_shape collision_size collision_xyz:='0 0 0'">
-        <link name="${name}">
+    <!-- ========== ARGUMENTS & PARAMETERS ========== -->
+    <xacro:arg name = "agent_name" default = "agent"/>
+    <xacro:arg name = "use_ros_control" default = "false"/>
+    <xacro:property name = "prefix" value = "$(arg agent_name)"/>
+    <xacro:property name = "wheel_effort" value = "1.0"/>
+    <!-- TODO - also change this in the controllers YAML file -->
+    <xacro:property name = "wheel_max_vel" value = "50.0"/>
+    <!-- ========== COMMON MACROS ========== -->
+    <xacro:macro name="common_link" params="prefix name material *origin collision_shape collision_size collision_xyz:='0 0 0'">
+        <link name="${prefix}_${name}">
             <visual>
                 <geometry>
@@ -25,18 +32,18 @@
         </link>
     </xacro:macro>
-    <xacro:macro name="continuous_joint" params="name parent child xyz rpy axis">
-        <joint name="${name}" type="continuous">
-            <parent link="${parent}"/>
-            <child link="${child}"/>
+    <xacro:macro name="continuous_joint" params="prefix name parent child xyz rpy axis">
+        <joint name="${prefix}_${name}" type="continuous">
+            <parent link="${prefix}_${parent}"/>
+            <child link="${prefix}_${child}"/>
             <origin xyz="${xyz}" rpy="${rpy}"/>
             <axis xyz="${axis}"/>
-            <limit lower="${-pi}" upper="${pi}" effort="100" velocity="2.5"/>
+            <limit effort="${wheel_effort}" velocity="${wheel_max_vel}"/>
             <dynamics friction="1E-04"/>
         </joint>
     </xacro:macro>
-    <xacro:macro name="fixed_joint" params="name parent child xyz rpy">
-        <joint name="${name}" type="fixed">
-            <parent link="${parent}"/>
-            <child link="${child}"/>
+    <xacro:macro name="fixed_joint" params="prefix name parent child xyz rpy">
+        <joint name="${prefix}_${name}" type="fixed">
+            <parent link="${prefix}_${parent}"/>
+            <child link="${prefix}_${child}"/>
             <origin xyz="${xyz}" rpy="${rpy}"/>
         </joint>
@@ -55,3 +62,12 @@
     <xacro:include filename = "x3_body.xacro"/>
     <xacro:include filename = "x3_sensors.xacro"/>
+    <xacro:include filename = "x3_gazebo_properties.xacro"/>
+    <!-- if using ros2_control -->
+    <xacro:if value = "$(arg use_ros_control)">
+        <xacro:include filename = "x3_ros_control.xacro"/>
+    </xacro:if>
+    <!-- if using gazebo control -->
+    <xacro:unless value = "$(arg use_ros_control)">
+        <xacro:include filename = "x3_gazebo_control.xacro"/>
+    </xacro:unless>
 </robot>

File: src/x3_description/urdf/x3_body.xacro (robot description, xacro)
@@ -9,6 +9,6 @@
     </material>
     <!-- Base links -->
-    <link name="base_footprint"/>
-    <xacro:common_link name="base_link" material="Green" collision_shape="box" collision_size="0.2235 0.139 0.1165" collision_xyz='0.005 0 0.0025    '>
+    <link name="${prefix}_base_footprint"/>
+    <xacro:common_link prefix="${prefix}" name="base_link" material="Green" collision_shape="box" collision_size="0.2235 0.139 0.1165" collision_xyz='0.005 0 0.0025    '>
         <inertial>
             <origin xyz="0.00498197982182523 5.70233829969297E-05 -0.0121008098068578" rpy="0 0 0"/>
@@ -24,9 +24,9 @@
     </xacro:common_link>
     <!-- Fixed Joints -->
-    <xacro:fixed_joint name="base_joint" parent="base_footprint" child="base_link" xyz="0.0 0.0 0.0850" rpy="0 0 0"/>
-    <link name="imu_link"/>
-    <xacro:fixed_joint name="base_imu" parent="base_link" child="imu_link" xyz="-0.06 0.025 0.095" rpy="0 3.1415 1.5707"/>
+    <xacro:fixed_joint prefix="${prefix}" name="base_joint" parent="base_footprint" child="base_link" xyz="0.0 0.0 0.0850" rpy="0 0 0"/>
+    <link name="${prefix}_imu_link"/>
+    <xacro:fixed_joint prefix="${prefix}" name="base_imu" parent="base_link" child="imu_link" xyz="-0.06 0.025 0.095" rpy="0 3.1415 1.5707"/>
     <!-- Wheels -->
-    <xacro:common_link name="front_right_wheel" material="White" collision_shape="cylinder" collision_size="0.035 0.03">
+    <xacro:common_link prefix="${prefix}" name="front_right_wheel" material="White" collision_shape="cylinder" collision_size="0.035 0.03">
         <inertial>
             <origin xyz="1.9051E-06 -2.3183E-07 -0.00064079" rpy="0 0 0"/>
@@ -36,7 +36,6 @@
         </inertial>
     </xacro:common_link>
-    <xacro:continuous_joint name="front_right_joint" parent="base_link" child="front_right_wheel"
-                      xyz="0.08 -0.0845 -0.0389" rpy="-${pi/2} 0 0" axis="0 0 1"/>
-    <xacro:common_link name="front_left_wheel" material="White" collision_shape="cylinder" collision_size="0.035 0.03">
+    <xacro:continuous_joint prefix="${prefix}" name="front_right_joint" parent="base_link" child="front_right_wheel" xyz="0.08 -0.0845 -0.0389" rpy="${pi/2} 0 0" axis="0 0 -1"/>
+    <xacro:common_link prefix="${prefix}" name="front_left_wheel" material="White" collision_shape="cylinder" collision_size="0.035 0.03">
         <inertial>
             <origin xyz="2.3728E-06 -9.4228E-07 0.00064068" rpy="0 0 0"/>
@@ -46,7 +45,6 @@
         </inertial>
     </xacro:common_link>
-    <xacro:continuous_joint name="front_left_joint" parent="base_link" child="front_left_wheel"
-                      xyz="0.08 0.0845 -0.0389" rpy="${pi/2} 0 0" axis="0 0 -1"/>
-    <xacro:common_link name="back_right_wheel" material="White" collision_shape="cylinder" collision_size="0.035 0.03">
+    <xacro:continuous_joint prefix="${prefix}" name="front_left_joint" parent="base_link" child="front_left_wheel" xyz="0.08 0.0845 -0.0389" rpy="${pi/2} 0 0" axis="0 0 -1"/>
+    <xacro:common_link prefix="${prefix}" name="back_right_wheel" material="White" collision_shape="cylinder" collision_size="0.035 0.03">
         <inertial>
             <origin xyz="-1.75924169923403E-06 1.28388821071107E-06 -0.000590549296238266" rpy="0 0 0"/>
@@ -56,7 +54,6 @@
         </inertial>
     </xacro:common_link>
-    <xacro:continuous_joint name="back_right_joint" parent="base_link" child="back_right_wheel"
-                      xyz="-0.08 -0.0845 -0.0395" rpy="-${pi/2} 0 0" axis="0 0 1"/>
-    <xacro:common_link name="back_left_wheel" material="White" collision_shape="cylinder" collision_size="0.035 0.03">
+    <xacro:continuous_joint prefix="${prefix}" name="back_right_joint" parent="base_link" child="back_right_wheel" xyz="-0.08 -0.0845 -0.0395" rpy="${pi/2} 0 0" axis="0 0 -1"/>
+    <xacro:common_link prefix="${prefix}" name="back_left_wheel" material="White" collision_shape="cylinder" collision_size="0.035 0.03">
         <inertial>
             <origin xyz="-4.01213085227115E-07 2.04910264598596E-06 0.000590775697051377" rpy="0 0 0"/>
@@ -66,5 +63,4 @@
         </inertial>
     </xacro:common_link>
-    <xacro:continuous_joint name="back_left_joint" parent="base_link" child="back_left_wheel"
-                      xyz="-0.08 0.0845 -0.0395" rpy="${pi/2} 0 0" axis="0 0 -1"/>
+    <xacro:continuous_joint prefix="${prefix}" name="back_left_joint" parent="base_link" child="back_left_wheel" xyz="-0.08 0.0845 -0.0395" rpy="${pi/2} 0 0" axis="0 0 -1"/>
 </robot>

File: src/x3_description/urdf/x3_sensors.xacro (robot description, xacro)
@@ -3,5 +3,5 @@
     <!-- PERIPHERALS -->
     <!-- lidar -->
-    <link name = "lidar_link">
+    <link name = "${prefix}_lidar_link">
         <visual>
             <origin xyz = "0 0 0" rpy = "1.570796 0 ${1.570796 - pi}"/>
@@ -26,7 +26,7 @@
         </inertial>
     </link>
-    <xacro:fixed_joint name="lidar_joint" parent="base_link" child="lidar_link" xyz="0.0405 5.25826986680105E-05 0.08285" rpy="0 0 ${pi}"/>
+    <xacro:fixed_joint prefix="${prefix}" name="lidar_joint" parent="base_link" child="lidar_link" xyz="0.0405 5.25826986680105E-05 0.08285" rpy="0 0 0"/>
     <!-- camera -->
-    <xacro:common_link name="camera_link" material="White" collision_shape="box" collision_size="0.06 0.17 0.05">
+    <xacro:common_link prefix="${prefix}" name="camera_link" material="White" collision_shape="box" collision_size="0.06 0.17 0.05">
         <inertial>
             <origin xyz="0 0 0" rpy="0 0 0"/>
@@ -35,7 +35,7 @@
         </inertial>
     </xacro:common_link>
-    <xacro:fixed_joint name="camera_joint" parent="base_link" child="camera_link" xyz="0.085105 1.7948E-05 0.06" rpy="0 -0.415 0"/>
+    <xacro:fixed_joint prefix="${prefix}" name="camera_joint" parent="base_link" child="camera_link" xyz="0.085105 1.7948E-05 0.06" rpy="0 -0.415 0"/>
     <!-- Optical camera link & joint -->
-    <link name="camera_link_optical"></link>
-    <xacro:fixed_joint name="camera_optical_joint" parent="camera_link" child="camera_link_optical" xyz="0 0 0" rpy="-${pi/2} 0 -${pi/2}"/>
+    <link name="${prefix}_camera_link_optical"></link>
+    <xacro:fixed_joint prefix="${prefix}" name="camera_optical_joint" parent="camera_link" child="camera_link_optical" xyz="0 0 0" rpy="-${pi/2} 0 -${pi/2}"/>
 </robot>
