Commit message: [x3_bringup & x3_description] fold the static tf of the LiDAR into the URDF
- the LiDAR scans are now rotated correctly
- the physical lidar link has the correct orientation in rviz

File: src/x3_description/urdf/x3_sensors.xacro (robot description, xacro)
@@ -5,5 +5,5 @@
     <link name = "lidar_link">
         <visual>
-            <origin xyz = "0 0 0" rpy = "1.570796 0 1.570796"/>
+            <origin xyz = "0 0 0" rpy = "1.570796 0 ${1.570796 - pi}"/>
             <geometry>
                 <mesh filename = "package://x3_description/meshes/lidar_link.STL" scale = "0.001 0.001 0.001"/>
@@ -26,5 +26,5 @@
         </inertial>
     </link>
-    <xacro:fixed_joint name="lidar_joint" parent="base_link" child="lidar_link" xyz="0.0405 5.25826986680105E-05 0.08285" rpy="0 0 0"/>
+    <xacro:fixed_joint name="lidar_joint" parent="base_link" child="lidar_link" xyz="0.0405 5.25826986680105E-05 0.08285" rpy="0 0 ${pi}"/>
     <!-- camera -->
     <xacro:common_link name="camera_link" material="White" collision_shape="box" collision_size="0.06 0.17 0.05">
