Commit message: [x3_description/drl_policy/apf_planner] rotate the lidar visual instead of the joint since it had negative impact on the rf2o scan matching

File: src/x3_description/urdf/x3_sensors.xacro (robot description, xacro)
@@ -5,5 +5,5 @@
     <link name = "${prefix}_lidar_link">
         <visual>
-            <origin xyz = "0 0 0" rpy = "1.570796 0 ${1.570796 - pi}"/>
+            <origin xyz = "0 0 0" rpy = "${pi/2} 0 ${pi/2}"/>
             <geometry>
                 <mesh filename = "package://x3_description/meshes/lidar_link.STL" scale = "0.001 0.001 0.001"/>
@@ -26,5 +26,5 @@
         </inertial>
     </link>
-    <xacro:fixed_joint prefix="${prefix}" name="lidar_joint" parent="base_link" child="lidar_link" xyz="0.0405 5.25826986680105E-05 0.08285" rpy="0 0 ${pi}"/>
+    <xacro:fixed_joint prefix="${prefix}" name="lidar_joint" parent="base_link" child="lidar_link" xyz="0.0405 5.25826986680105E-05 0.08285" rpy="0 0 0"/>
     <!-- camera -->
     <xacro:common_link prefix="${prefix}" name="camera_link" material="White" collision_shape="box" collision_size="0.06 0.17 0.05">
